File: Lab1.sch (KiCad schematic (older format))
At the start: 21 parts, among them J1 USB_OTG, J2 SWD connector, U1 LM1117ADJ, U2 CMWX1ZZABZ-078

Commit message: Finished Lab2 Layout
Parts:
- U1: symbol E7020E:LM1117ADJ -> Lab1-rescue:LM1117ADJ-E7020E
- U2: footprint CMWX177AB7:CMWX1ZZABZ -> CMWX177AB7:CMWX1ZZABZ_longer_pads
Changed lines of the file:
@@
 F 0 "U2" H 5900 2514 50  0000 C CNN
 F 1 "CMWX1ZZABZ-078" H 5900 2423 50  0000 C CNN
-F 2 "CMWX177AB7:CMWX1ZZABZ" H 5900 4100 50  0001 C CNN
+F 2 "CMWX177AB7:CMWX1ZZABZ_longer_pads" H 5900 4100 50  0001 C CNN
 F 3 "https://wireless.murata.com/RFM/data/type_abz.pdf" H 8350 2600 50  0001 C CNN
 	1    5900 4100
@@
 $EndComp
 $Comp
-L E7020E:LM1117ADJ U1
+L Lab1-rescue:LM1117ADJ-E7020E U1
 U 1 1 5E2DB034
 P 3150 2050
